Commit message: gripper added to the robot model

File: urdf/kobuki.urdf.xacro (robot description, xacro)
@@ -7,6 +7,6 @@
  -->
 <robot name="kobuki" xmlns:xacro="http://ros.org/wiki/xacro">
-  <xacro:include filename="$(find robot_arm_simulator)/urdf/common_properties.urdf.xacro"/>
-  <xacro:include filename="$(find robot_arm_simulator)/urdf/kobuki_gazebo.urdf.xacro"/>
+  <xacro:include filename="$(find hola_tortuga)/urdf/common_properties.urdf.xacro"/>
+  <xacro:include filename="$(find hola_tortuga)/urdf/kobuki_gazebo.urdf.xacro"/>
   <!-- Kobuki -->
   <xacro:macro name="kobuki">
@@ -292,10 +292,9 @@
       </collision>
     </link>
-    <joint name="arm_joint_4" type="prismatic">
+    <joint name="arm_joint_4" type="fixed">
       <parent link="arm_link_3"/>
       <child link="arm_link_4"/>
-      <origin xyz="0.0 0.0 0.11"/>
+      <origin xyz="0.0 0.0 0.13"/>
       <axis xyz="0 0 1"/>
-      <limit effort="1000" lower="-0.10" upper="0.06" velocity="5"/>
     </joint>
     <link name="arm_link_4">
@@ -312,4 +311,48 @@
         </geometry>
         <origin xyz="0.0 0.0 0.05"/>
+      </collision>
+    </link>
+    <joint name="arm_joint_L" type="prismatic">
+      <parent link="arm_link_4"/>
+      <child link="arm_link_L"/>
+      <origin xyz="0.0 0.005 0.0"/>
+      <axis xyz="0 1 0"/>
+      <limit effort="100" lower="0.0" upper="0.03" velocity="5"/>
+    </joint>
+    <link name="arm_link_L">
+      <visual>
+        <geometry>
+          <box size="0.02 0.01 0.04"/>
+        </geometry>
+        <origin xyz="0.0 0.0 0.03"/>
+        <material name="blue"/>
+      </visual>
+      <collision>
+        <geometry>
+          <box size="0.02 0.01 0.04"/>
+        </geometry>
+        <origin xyz="0.0 0.0 0.03"/>
+      </collision>
+    </link>
+    <joint name="arm_joint_R" type="prismatic">
+      <parent link="arm_link_4"/>
+      <child link="arm_link_R"/>
+      <origin xyz="0.0 -0.005 0.0"/>
+      <axis xyz="0 -1 0"/>
+      <limit effort="100" lower="0.0" upper="0.03" velocity="5"/>
+    </joint>
+    <link name="arm_link_R">
+      <visual>
+        <geometry>
+          <box size="0.02 0.01 0.04"/>
+        </geometry>
+        <origin xyz="0.0 0.0 0.03"/>
+        <material name="blue"/>
+      </visual>
+      <collision>
+        <geometry>
+          <box size="0.02 0.01 0.04"/>
+        </geometry>
+        <origin xyz="0.0 0.0 0.03"/>
       </collision>
     </link>

Commit message: Servicio para mover el brazo

File: urdf/kobuki.urdf.xacro (robot description, xacro)
@@ -167,5 +167,5 @@
     </material>
     <joint name="arm_base_joint" type="fixed">
-      <origin xyz="0 0 0.089" rpy="0 0 0" />
+      <origin xyz="0.065 0 0.089" rpy="0 0 0" />
       <parent link="base_link"/>
       <child link="arm_base_link" />
@@ -174,12 +174,12 @@
       <visual>
         <geometry>
-          <cylinder length="0.08" radius="0.07"/>
-        </geometry>
-        <origin xyz="0.0 0.0 0.04"/>
+          <cylinder length="0.05" radius="0.07"/>
+        </geometry>
+        <origin xyz="0.0 0.0 0.025"/>
         <material name="blue"/>
       </visual>
       <collision>
         <geometry>
-          <cylinder length="0.1" radius="0.4"/>
+          <cylinder length="0.05" radius="0.07"/>
         </geometry>
         <origin xyz="0.0 0.0 0.025"/>
@@ -190,5 +190,5 @@
       <parent link="arm_base_link"/>
       <child link="arm_link_0"/>
-      <origin xyz="0.0 0.0 0.08"/>
+      <origin xyz="0.0 0.0 0.05"/>
       <axis xyz="0 0 1"/>
       <limit effort="1000" lower="-3.14" upper="3.14" velocity="5"/>

Commit message: Se mejora la visualización del problema, se documenta el launch y se organiza mejor para evitar reescritura de código.

File: urdf/kobuki.urdf.xacro (robot description, xacro)
@@ -10,4 +10,5 @@
   <xacro:include filename="$(find hola_tortuga)/urdf/common_properties.urdf.xacro"/>
   <xacro:include filename="$(find hola_tortuga)/urdf/kobuki_gazebo.urdf.xacro"/>
+  <xacro:include filename="$(find hola_tortuga)/urdf/kobuki_arm.urdf.xacro"/>
   <!-- Kobuki -->
   <xacro:macro name="kobuki">
@@ -152,5 +153,6 @@
     </link>
     <!-- Kobuki's arm -->
-    <material name="blue">
+    <kobuki_arm parent="base_link"/>
+    <!-- <material name="blue">
       <color rgba="0 0 1 1"/>
     </material>
@@ -357,5 +359,5 @@
         <origin xyz="0.0 0.0 0.03"/>
       </collision>
-    </link>
+    </link>  -->
     <!---->
     <!-- Kobuki's sensors -->
